Commit message: Added lolo prefab

File: Runtime/URDF/lolo/rviz.xacro (robot description, xacro)
@@ -1,12 +1,12 @@
 <?xml version="1.0"?>
 <robot name="lolo_auv" xmlns:xacro="http://www.ros.org/wiki/xacro">
-  <xacro:property name="visual_mesh_file" value="file://$(find lolo_description)/mesh/lolo_hull.dae"/>
-  <xacro:property name="prop_port_mesh_file" value="file://$(find lolo_description)/mesh/lolo_port_propeller.dae"/>
-  <xacro:property name="prop_strb_mesh_file" value="file://$(find lolo_description)/mesh/lolo_strb_propeller.dae"/>
-  <xacro:property name="rudder_mesh_file" value="file://$(find lolo_description)/mesh/lolo_rudder.dae"/>
-  <xacro:property name="elevon_port_mesh_file" value="file://$(find lolo_description)/mesh/lolo_port_elevon.dae"/>
-  <xacro:property name="elevon_strb_mesh_file" value="file://$(find lolo_description)/mesh/lolo_strb_elevon.dae"/>
-  <xacro:property name="elevator_mesh_file" value="file://$(find lolo_description)/mesh/lolo_elevator.dae"/>
-  <link name="$(arg robot_namespace)/base_link">
+  <xacro:property name="visual_mesh_file" value="mesh/lolo_hull.dae"/>
+  <xacro:property name="prop_port_mesh_file" value="mesh/lolo_port_propeller.dae"/>
+  <xacro:property name="prop_strb_mesh_file" value="mesh/lolo_strb_propeller.dae"/>
+  <xacro:property name="rudder_mesh_file" value="mesh/lolo_rudder.dae"/>
+  <xacro:property name="elevon_port_mesh_file" value="mesh/lolo_port_elevon.dae"/>
+  <xacro:property name="elevon_strb_mesh_file" value="mesh/lolo_strb_elevon.dae"/>
+  <xacro:property name="elevator_mesh_file" value="mesh/lolo_elevator.dae"/>
+  <link name="base_link">
     <visual>
       <origin xyz="0 0 0" rpy="0 0 0"/>
@@ -16,13 +16,13 @@
     </visual>
   </link>
-  <link name="$(arg robot_namespace)/dvl_link"/>
-  <link name="$(arg robot_namespace)/compass_link"/>
-  <link name="$(arg robot_namespace)/fls_link"/>
-  <link name="$(arg robot_namespace)/imu_link"/>
-  <link name="$(arg robot_namespace)/pressure_link"/>
-  <link name="$(arg robot_namespace)/gps_link"/>
-  <link name="$(arg robot_namespace)/mbes_link"/>
-  <link name="$(arg robot_namespace)/usbl_link"/>
-  <link name="$(arg robot_namespace)/elevator">
+  <link name="dvl_link"/>
+  <link name="compass_link"/>
+  <link name="fls_link"/>
+  <link name="imu_link"/>
+  <link name="pressure_link"/>
+  <link name="gps_link"/>
+  <link name="mbes_link"/>
+  <link name="usbl_link"/>
+  <link name="elevator">
     <visual>
       <origin xyz="0 0 0" rpy="0 0 0" />
@@ -32,5 +32,5 @@
     </visual>
   </link>
-  <link name="$(arg robot_namespace)/rudder_stbd">
+  <link name="rudder_stbd">
     <visual>
       <origin xyz="0 0 0" rpy="0 0 0" />
@@ -40,5 +40,5 @@
     </visual>
   </link>
-  <link name="$(arg robot_namespace)/rudder_port">
+  <link name="rudder_port">
     <visual>
       <origin xyz="0 0 0" rpy="0 0 0" />
@@ -48,5 +48,5 @@
     </visual>
   </link>
-  <link name="$(arg robot_namespace)/elevon_stbd">
+  <link name="elevon_stbd">
     <visual>
       <origin xyz="0 0 0" rpy="0 0 0" />
@@ -56,5 +56,5 @@
     </visual>
   </link>
-  <link name="$(arg robot_namespace)/elevon_port">
+  <link name="elevon_port">
     <visual>
       <origin xyz="0 0 0" rpy="0 0 0" />
@@ -64,5 +64,5 @@
     </visual>
   </link>
-  <link name="$(arg robot_namespace)/thruster_port">
+  <link name="thruster_port">
     <visual>
       <origin xyz="0.0 0 0" rpy="0 0 0" />
@@ -72,5 +72,5 @@
     </visual>
   </link>
-  <link name="$(arg robot_namespace)/thruster_stbd">
+  <link name="thruster_stbd">
     <visual>
       <origin xyz="0.0 0 0" rpy="0 0 0" />
@@ -81,5 +81,5 @@
   </link>
   <!-- Mount a 3D pose sensor -->
-  <link name="$(arg robot_namespace)/pose_sensor_link">
+  <link name="pose_sensor_link">
     <visual>
       <geometry>
@@ -88,97 +88,97 @@
     </visual>
   </link>
-  <joint name="$(arg robot_namespace)/elevator_joint" type="revolute">
+  <joint name="elevator_joint" type="revolute">
     <origin xyz="-0.6476 0.0 0.0135" rpy="0 0 0" />
-    <parent link="$(arg robot_namespace)/base_link" />
-    <child link="$(arg robot_namespace)/elevator" />
+    <parent link="base_link" />
+    <child link="elevator" />
     <limit effort="0" lower="-${pi/4.0}" upper="${pi/4.0}" velocity="0"/>
     <axis xyz="0 1 0"/>
   </joint>
-  <joint name="$(arg robot_namespace)/rudder_stbd_joint" type="revolute">
+  <joint name="rudder_stbd_joint" type="revolute">
     <origin xyz="-0.3278 -0.253 0.129" rpy="0 0 0" />
-    <parent link="$(arg robot_namespace)/base_link" />
-    <child link="$(arg robot_namespace)/rudder_stbd" />
+    <parent link="base_link" />
+    <child link="rudder_stbd" />
     <limit effort="0" lower="-${pi/4.0}" upper="${pi/4.0}" velocity="0"/>
     <axis xyz="0 0 1"/>
   </joint>
-  <joint name="$(arg robot_namespace)/rudder_port_joint" type="revolute">
+  <joint name="rudder_port_joint" type="revolute">
     <origin xyz="-0.3278 0.253 0.129" rpy="0 0 0" />
-    <parent link="$(arg robot_namespace)/base_link" />
-    <child link="$(arg robot_namespace)/rudder_port" />
+    <parent link="base_link" />
+    <child link="rudder_port" />
     <limit effort="0" lower="-${pi/4.0}" upper="${pi/4.0}" velocity="0"/>
     <axis xyz="0 0 1"/>
   </joint>
-  <joint name="$(arg robot_namespace)/elevon_stbd_joint" type="revolute">
+  <joint name="elevon_stbd_joint" type="revolute">
     <origin xyz="-0.3733 -0.4035 0.01349" rpy="0 0 -0.19652" />
-    <parent link="$(arg robot_namespace)/base_link" />
-    <child link="$(arg robot_namespace)/elevon_stbd" />
+    <parent link="base_link" />
+    <child link="elevon_stbd" />
     <limit effort="0" lower="-${pi/4.0}" upper="${pi/4.0}" velocity="0"/>
     <axis xyz="0 1 0"/>
   </joint>
-  <joint name="$(arg robot_namespace)/elevon_port_joint" type="revolute">
+  <joint name="elevon_port_joint" type="revolute">
     <origin xyz="-0.3733 0.4035 0.01349" rpy="0 0 0.19652" />
-    <parent link="$(arg robot_namespace)/base_link" />
-    <child link="$(arg robot_namespace)/elevon_port" />
+    <parent link="base_link" />
+    <child link="elevon_port" />
     <limit effort="0" lower="-${pi/4.0}" upper="${pi/4.0}" velocity="0"/>
     <axis xyz="0 1 0"/>
   </joint>
   <!-- Propeller -->
-  <joint name="$(arg robot_namespace)/thruster_stbd_joint" type="continuous">
+  <joint name="thruster_stbd_joint" type="continuous">
     <origin xyz="-0.9056 -0.2754 0.013678" rpy="0 0 0" />
     <axis xyz="1 0 0"/>
-    <parent link="$(arg robot_namespace)/base_link"/>
-    <child link="$(arg robot_namespace)/thruster_stbd"/>
+    <parent link="base_link"/>
+    <child link="thruster_stbd"/>
   </joint>
-  <joint name="$(arg robot_namespace)/thruster_port_joint" type="continuous">
+  <joint name="thruster_port_joint" type="continuous">
     <origin xyz="-0.9056 0.2754 0.013678" rpy="0 0 0" />
     <axis xyz="1 0 0"/>
-    <parent link="$(arg robot_namespace)/base_link"/>
-    <child link="$(arg robot_namespace)/thruster_port"/>
+    <parent link="base_link"/>
+    <child link="thruster_port"/>
   </joint>
-  <joint name="$(arg robot_namespace)/pose_sensor_joint" type="revolute">
+  <joint name="pose_sensor_joint" type="revolute">
     <origin xyz="0 0 0" rpy="0 0 0" />
-    <parent link="$(arg robot_namespace)/base_link"/>
-    <child link="$(arg robot_namespace)/pose_sensor_link"/>
+    <parent link="base_link"/>
+    <child link="pose_sensor_link"/>
     <limit effort="0" lower="0" upper="0" velocity="0"/>
   </joint>
-  <joint name="$(arg robot_namespace)/dvl_joint" type="fixed">
+  <joint name="dvl_joint" type="fixed">
     <origin xyz="0.805 -0.025 -0.245" rpy="3.14159 0 0" />
-    <parent link="$(arg robot_namespace)/base_link"/>
-    <child link="$(arg robot_namespace)/dvl_link"/>
+    <parent link="base_link"/>
+    <child link="dvl_link"/>
   </joint>
-  <joint name="$(arg robot_namespace)/compass_joint" type="fixed">
+  <joint name="compass_joint" type="fixed">
     <origin xyz="0 0 0" rpy="0 0 0" />
-    <parent link="$(arg robot_namespace)/base_link"/>
-    <child link="$(arg robot_namespace)/compass_link"/>
+    <parent link="base_link"/>
+    <child link="compass_link"/>
   </joint>
-  <joint name="$(arg robot_namespace)/fls_joint" type="fixed">
+  <joint name="fls_joint" type="fixed">
     <origin xyz="0 0 0" rpy="0 0 0" />
-    <parent link="$(arg robot_namespace)/base_link"/>
-    <child link="$(arg robot_namespace)/fls_link"/>
+    <parent link="base_link"/>
+    <child link="fls_link"/>
   </joint>
-  <joint name="$(arg robot_namespace)/imu_joint" type="fixed">
+  <joint name="imu_joint" type="fixed">
     <origin xyz="0 0 0" rpy="3.14159 0 0" />
-    <parent link="$(arg robot_namespace)/base_link"/>
-    <child link="$(arg robot_namespace)/imu_link"/>
+    <parent link="base_link"/>
+    <child link="imu_link"/>
   </joint>
-  <joint name="$(arg robot_namespace)/pressure_joint" type="fixed">
+  <joint name="pressure_joint" type="fixed">
     <origin xyz="0 0 0" rpy="0 0 0" />
-    <parent link="$(arg robot_namespace)/base_link"/>
-    <child link="$(arg robot_namespace)/pressure_link"/>
+    <parent link="base_link"/>
+    <child link="pressure_link"/>
   </joint>
-  <joint name="$(arg robot_namespace)/gps_joint" type="fixed">
+  <joint name="gps_joint" type="fixed">
     <origin xyz="0.836 0 0.44" rpy="0 0 0" />
-    <parent link="$(arg robot_namespace)/base_link"/>
-    <child link="$(arg robot_namespace)/gps_link"/>
+    <parent link="base_link"/>
+    <child link="gps_link"/>
   </joint>
-  <joint name="$(arg robot_namespace)/mbes_joint" type="fixed">
+  <joint name="mbes_joint" type="fixed">
     <origin xyz="2.523 0.0155 -0.302" rpy="3.14159 1.53589 0" />
-    <parent link="$(arg robot_namespace)/base_link"/>
-    <child link="$(arg robot_namespace)/mbes_link"/>
+    <parent link="base_link"/>
+    <child link="mbes_link"/>
   </joint>
-  <joint name="$(arg robot_namespace)/usbl_joint" type="fixed">
+  <joint name="usbl_joint" type="fixed">
     <origin xyz="0.389 0.002 0.337" rpy="0 0 0" />
-    <parent link="$(arg robot_namespace)/base_link"/>
-    <child link="$(arg robot_namespace)/usbl_link"/>
+    <parent link="base_link"/>
+    <child link="usbl_link"/>
   </joint>
 </robot>
