Commit message: WIP

File: Runtime/URDF/sam_auv/sam_auv.urdf (robot description, URDF)
Before this commit: robot sam_auv, 19 links, 18 joints
Links:
- added link vbs_link, mass 0.150
Joints:
- added joint vbs_joint: type prismatic, parent base_link, child vbs_link, origin xyz=-0.245 0 -0.012 rpy=0.0 0.0 0.0, axis 1 0 0, limit lower=-0.058 upper=0 effort=1.0 velocity=0.2
- joint lcg_joint: limit lower=-0.03 upper=0.03 effort=1.0 velocity=0.2 -> lower=-0.030 upper=0.030 effort=1.0 velocity=0.2

Commit message: Fixed VBS

File: Runtime/URDF/sam_auv/sam_auv.urdf (robot description, URDF)
Before this commit: robot sam_auv, 20 links, 19 joints
Links:
- link base_link: mass 12.35 -> 12.29
- link vbs_link: mass 0.150 -> 0.300

Commit message: Mass change in line with force feedback

File: Runtime/URDF/sam_auv/sam_auv.urdf (robot description, URDF)
Before this commit: robot sam_auv, 20 links, 19 joints
Links:
- link base_link: mass 12.29 -> 12.317
- link vbs_link: mass 0.300 -> 0.24925

Commit message: Proper import structure

File: Runtime/URDF/sam_auv/sam_auv.urdf (robot description, URDF)
Before this commit: robot sam_auv, 20 links, 19 joints
Links:
- link base_link: mass 12.317 -> 12.012
Joints:
- joint lcg_joint: axis 1 0 0 -> -1 0 0; limit lower=-0.030 upper=0.030 effort=1.0 velocity=0.2 -> lower=0 upper=0.057 effort=1.0 velocity=0.2; origin xyz=0.083 0.0 0.0 rpy=0.0 0.0 0.0 -> xyz=-0.08 0.0 0.0 rpy=0.0 0.0 0.0
- joint vbs_joint: limit lower=-0.058 upper=0 effort=1.0 velocity=0.2 -> lower=0.006 upper=0.05 effort=1.0 velocity=0.2; origin xyz=-0.245 0 -0.012 rpy=0.0 0.0 0.0 -> xyz=-0.273 0 -0.0125 rpy=0.0 0.0 0.0
